File: PCB/Boost.kicad_sch (KiCad schematic)
At the start: 24 parts, among them IC1 MC34063ADR, Q1 BSS84, U1 AMS1117-3.3

Commit message: Firmware initial commit
Changed lines of the file:
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@@
+	)
+	(junction
+		(at 63.5 91.44)
+		(diameter 0)
+		(color 0 0 0 0)
 	)
 	(junction
@@
 	)
 	(junction
-		(at 63.5 91.44)
-		(diameter 0)
-		(color 0 0 0 0)
-	)
-	(junction
 		(at 199.39 67.31)
 		(diameter 0)
@@
 	(wire
 		(pts
-			(xy 54.61 91.44) (xy 63.5 91.44)
+			(xy 57.15 91.44) (xy 63.5 91.44)
 		)
 		(stroke
@@
 	(hierarchical_label "BATT_{IN}"
 		(shape input)
-		(at 54.61 91.44 180)
-		(effects
-			(font
+		(at 57.15 91.44 180)
+		(effects
+			(font
