File: PCB/Boost.kicad_sch (KiCad schematic)
At the start: 24 parts, among them IC1 MC34063ADR, Q1 BSS84, U1 AMS1117-3.3

Commit message: Initial Commit for INA219
Parts:
- removed R27: 5.1k, Resistor_SMD:R_0402_1005Metric, symbol Device:R
- removed R28: 10k, Resistor_SMD:R_0402_1005Metric, symbol Device:R
- D2: value D -> SS12; footprint (none) -> Diode_SMD:D_SMA
- R3: value 3k3 -> 10k
- R4: value 10k -> 39k
Connections:
- net BATT_{IN} renamed V_{IN}
- net V_{BATT} renamed V_{SYS}
Other:
- note added: "VOut = 1.25(1+R4/R3)= 6.1"
- note removed: "VOut = 1.25(1+R4/R3)= 5"

Commit message: V2.1
Other:
- note added: "220m"
- note removed: "22m"
Changed lines of the file:
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@@
 		)
 	)
-	(text "22m"
+	(text "220m"
 		(exclude_from_sim no)
 		(at 40.64 90.424 0)

Commit message: LIbrary Health
Parts:
- C6: footprint CAPPM7344X310N -> Footprints:TAJD337K010RNJ
- C8: footprint CAPPM3528X210N -> Footprints:TAJB226K020RNJ
- IC1: footprint SOIC127P600X175-8N -> Footprints:MC34063ADR
Changed lines of the file:
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@@
-	)
-	(junction
-		(at 63.5 91.44)
-		(diameter 0)
-		(color 0 0 0 0)
 	)
 	(junction
@@
 	)
 	(junction
+		(at 63.5 90.17)
+		(diameter 0)
+		(color 0 0 0 0)
+	)
+	(junction
 		(at 144.78 95.25)
 		(diameter 0)
@@
 	(wire
 		(pts
-			(xy 57.15 91.44) (xy 63.5 91.44)
+			(xy 52.07 90.17) (xy 63.5 90.17)
 		)
 		(stroke
@@
 	(wire
 		(pts
-			(xy 63.5 87.63) (xy 63.5 91.44)
+			(xy 63.5 87.63) (xy 63.5 90.17)
 		)
 		(stroke
@@
 	(wire
 		(pts
-			(xy 63.5 91.44) (xy 63.5 92.71)
+			(xy 63.5 90.17) (xy 63.5 92.71)
 		)
 		(stroke
@@
 	(hierarchical_label "V_{IN}"
 		(shape input)
-		(at 57.15 91.44 180)
+		(at 52.07 90.17 180)
 		(effects
 			(font
@@
 			)
 		)
-		(property "Footprint" "CAPPM3528X210N"
+		(property "Footprint" "Footprints:TAJB226K020RNJ"
 			(at 126.06 96.52 0)
 			(hide yes)
@@
 			)
 		)
-		(property "Footprint" "SOIC127P600X175-8N"
+		(property "Footprint" "Footprints:MC34063ADR"
 			(at 77.47 177.47 0)
 			(hide yes)
@@
 			)
 		)
-		(property "Footprint" "CAPPM7344X310N"
+		(property "Footprint" "Footprints:TAJD337K010RNJ"
 			(at 158.75 -37.77 0)
 			(hide yes)
