File: PCB/SolderCrateBox.kicad_sch (KiCad schematic)
At the start: 8 parts, among them J1 Conn_01x02, J2 Conn_01x02, J3 Conn_01x03, J4 Conn_01x03

Commit message: Firmware initial commit
Other:
- sheet ESP32 renamed ESP32_C3
Changed lines of the file:
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@@
 	(sheet
 		(at 101.6 37.465)
-		(size 17.78 53.34)
+		(size 17.78 36.195)
 		(exclude_from_sim no)
 		(in_bom yes)
@@
 			(color 0 0 0 0)
 		)
-		(property "Sheetname" "ESP32"
+		(property "Sheetname" "ESP32_C3"
 			(at 101.6 36.7534 0)
 			(show_name no)
@@
 		)
 		(property "Sheetfile" "ESP32.kicad_sch"
-			(at 101.6 91.3896 0)
+			(at 101.6 74.2446 0)
 			(show_name no)
 			(do_not_autoplace no)

Commit message: platformio commi
Other:
- note added: "ADD the INA current sensor for SoC calculation"
Changed lines of the file:
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@@
+		)
+	)
+	(text "ADD the INA current sensor for SoC calculation"
+		(exclude_from_sim no)
+		(at 76.962 72.898 0)
+		(effects
+			(font
+				(size 1.27 1.27)
+			)
 		)
 	)
@@
 	)
 	(label "LED.DATA"
-		(at 124.46 62.23 0)
-		(effects
-			(font
+		(at 125.73 62.23 0)
+		(effects
+			(font
