File: PCB/SolderCrateBox.kicad_sch (KiCad schematic)
At the start: 8 parts, among them J1 Conn_01x02, J2 Conn_01x02, J3 Conn_01x03, J4 Conn_01x03

Commit message: Initial Commit for INA219
Parts:
- added C11, C9: TAJE477K010RNJ, CAPPM7344X430N, symbol Capacitor_2:TAJE477K010RNJ
- J1, J2: footprint Connector_JST:JST_XH_B2B-XH-A_1x02_P2.50mm_Vertical -> Connector_JST:JST_PH_S2B-PH-K_1x02_P2.00mm_Horizontal
- J3, J4: footprint Connector_JST:JST_XH_S3B-XH-SM4-TB_1x03-1MP_P2.50mm_Horizontal -> Connector_JST:JST_PH_S3B-PH-K_1x03_P2.00mm_Horizontal
Connections:
- net GND: now also C11.2 (-), C9.2 (-)
- net +V_{BATT} renamed +V_{SYS}
- net +V_{SYS}: now also C11.1 (+), C9.1 (+)
- net Boost/BATT_{IN} renamed VI_Sensor/V_{In}
Other:
- added sheet VI_Sensor (VI_Sensor.kicad_sch)
- sheet Boost ports: added V_{IN}, V_{SYS}; removed BATT_{IN}, V_{BATT}, V_{Sense}
- note added: "470u"
- note removed: "ADD the INA current sensor for SoC calculation"
- moved on the sheet: C1, C2, J1, J2

Commit message: LIbrary Health
Parts:
- C11, C9: footprint CAPPM7344X430N -> Footprints:TAJE477K010RNJ
Connections:
- net VI_Sensor/V_{In} renamed VI_Sensor/INA_{IN}
Other:
- sheet VI_Sensor ports: added INA_{IN}, INA_{OUT}; removed V_{In}, V_{OUT}
Changed lines of the file:
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@@
 	(wire
 		(pts
-			(xy 53.34 33.02) (xy 62.23 33.02)
+			(xy 54.61 33.02) (xy 62.23 33.02)
 		)
 		(stroke
@@
 	(wire
 		(pts
-			(xy 53.34 50.8) (xy 53.34 33.02)
+			(xy 54.61 50.8) (xy 54.61 33.02)
 		)
 		(stroke
@@
 	(wire
 		(pts
-			(xy 53.34 50.8) (xy 52.07 50.8)
+			(xy 54.61 50.8) (xy 52.07 50.8)
 		)
 		(stroke
@@
 			)
 		)
-		(property "Footprint" "CAPPM7344X430N"
+		(property "Footprint" "Footprints:TAJE477K010RNJ"
 			(at 108.28 82.55 0)
 			(hide yes)
@@
 			)
 		)
-		(property "Footprint" "CAPPM7344X430N"
+		(property "Footprint" "Footprints:TAJE477K010RNJ"
 			(at 107.01 104.14 0)
 			(hide yes)
@@
 			)
 		)
-		(pin "V_{In}" input
+		(pin "SDA" input
+			(at 52.07 54.61 0)
+			(effects
+				(font
+					(size 1.27 1.27)
+				)
+				(justify right)
+			)
+		)
+		(pin "SCL" input
+			(at 52.07 57.15 0)
+			(effects
+				(font
+					(size 1.27 1.27)
+				)
+				(justify right)
+			)
+		)
+		(pin "INA_{IN}" input
 			(at 31.75 50.8 180)
 			(effects
@@
 			)
 		)
-		(pin "SDA" bidirectional
-			(at 52.07 54.61 0)
-			(effects
-				(font
-					(size 1.27 1.27)
-				)
-				(justify right)
-			)
-		)
-		(pin "V_{OUT}" output
+		(pin "INA_{OUT}" input
 			(at 52.07 50.8 0)
 			(effects
 				(font
-					(size 1.27 1.27)
-				)
-				(justify right)
-			)
-		)
-		(pin "SCL" bidirectional
-			(at 52.07 57.15 0)
-			(effects
-				(font
