File: PCB/ESP32.kicad_sch (KiCad schematic)
At the start: 15 parts, among them IC2 ESP32-C3-MINI-1U-N4X, J5 USB_C_Receptacle_USB2.0_16P, SW10 SW_Push, SW11 SW_Push, U2 USBLC6-2SC6

Commit message: LIbrary Health
Parts:
- IC2: footprint ESP32C3MINI1UN4X -> Footprints:ESP32C3MINI1UN4X
- J5: footprint Connector_USB:USB_C_Receptacle_G-Switch_GT-USB-7010ASV -> Footprints:USB_C_Receptacle_G-Switch_GT-USB-7010ASV
Changed lines of the file:
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@@
 			)
 		)
-		(property "Footprint" "Connector_USB:USB_C_Receptacle_G-Switch_GT-USB-7010ASV"
+		(property "Footprint" "Footprints:USB_C_Receptacle_G-Switch_GT-USB-7010ASV"
 			(at 54.61 49.53 0)
 			(hide yes)
@@
 			)
 		)
-		(property "Footprint" "ESP32C3MINI1UN4X"
+		(property "Footprint" "Footprints:ESP32C3MINI1UN4X"
 			(at 240.03 121.59 0)
 			(hide yes)
