File: PCB/VI_Sensor.kicad_sch (KiCad schematic)
At the start: 0 parts

Commit message: LIbrary Health
Parts:
- added C17: 100n, Capacitor_SMD:C_0402_1005Metric, symbol Device:C
- added IC5: INA219AIDR, Footprints:INA219AIDR, symbol Sensor_Current_2:INA219AIDR
- added R11: 0.01, Resistor_SMD:R_2512_6332Metric, symbol Device:R
- added R8, R9: 10k, Resistor_SMD:R_0402_1005Metric, symbol Device:R
Connections:
- new net +3V3: C17.1, IC5.5 (VS), R8.1, R9.1
- new net GND: C17.2, IC5.1 (A1), IC5.2 (A0), IC5.6 (GND)
- new net INA_{IN}: IC5.8 (IN+), R11.2
- new net INA_{OUT}: IC5.7 (IN-), R11.1
- new net SCL: IC5.4 (SCL), R8.2
- new net SDA: IC5.3 (SDA), R9.2
